File: drawings/Schematic.brd (EAGLE design)
At the start: 83.5 x 41.9 mm, 15 parts

Commit message: revise drawings
Connections:
- new net N$9: 2SC1815.3, R1.P$1
- net 5V: now also OPTO_PC817.4; no longer R1.P$2
- net GND: no longer OPTO_PC817.3
- net N$1: now also OPTO_PC817.3, R1.P$2; no longer 2SC1815.3, OPTO_PC817.4, R1.P$1
Routing:
- net 5V: track 59.4 -> 91.3 mm
- net 3.3V: track 61.4 -> 77.3 mm
- net N$1: track 11.3 -> 17.7 mm
- net N$9: track 0.00 -> 5.61 mm
- net GND: track 113.9 -> 118.6 mm
Changed lines of the file:
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@@
 <contactref element="USB" pad="VBUS1"/>
 <contactref element="D1" pad="C"/>
-<contactref element="R1" pad="P$2"/>
-<wire x1="19.05" y1="38.1" x2="40.64" y2="38.1" width="0.4064" layer="1"/>
-<wire x1="40.64" y1="38.1" x2="43.18" y2="35.56" width="0.4064" layer="1"/>
-<wire x1="43.18" y1="35.56" x2="46.99" y2="39.37" width="0.4064" layer="1"/>
-<wire x1="46.99" y1="39.37" x2="54.61" y2="39.37" width="0.4064" layer="1"/>
 <wire x1="54.61" y1="39.37" x2="58.42" y2="39.37" width="0.4064" layer="1"/>
 <wire x1="58.42" y1="39.37" x2="59.69" y2="38.1" width="0.4064" layer="1"/>
@@
 <wire x1="12.7" y1="36.83" x2="13.97" y2="38.1" width="0.4064" layer="1"/>
 <wire x1="13.97" y1="38.1" x2="19.05" y2="38.1" width="0.4064" layer="1"/>
+<contactref element="OPTO_PC817" pad="4"/>
+<wire x1="19.05" y1="38.1" x2="48.26" y2="38.1" width="0.4064" layer="1"/>
+<wire x1="48.26" y1="38.1" x2="49.53" y2="39.37" width="0.4064" layer="1"/>
+<wire x1="49.53" y1="39.37" x2="54.61" y2="39.37" width="0.4064" layer="1"/>
+<wire x1="45.8" y1="24.16" x2="62.26" y2="24.16" width="0.4064" layer="1"/>
+<wire x1="62.26" y1="24.16" x2="63.5" y2="25.4" width="0.4064" layer="1"/>
+<wire x1="63.5" y1="25.4" x2="63.5" y2="36.83" width="0.4064" layer="1"/>
+<wire x1="63.5" y1="36.83" x2="62.23" y2="38.1" width="0.4064" layer="1"/>
+<wire x1="62.23" y1="38.1" x2="59.69" y2="38.1" width="0.4064" layer="1"/>
 </signal>
 <signal name="3.3V">
@@
 <wire x1="12.7" y1="34.29" x2="12.7" y2="24.13" width="0.4064" layer="16"/>
 <wire x1="12.7" y1="24.13" x2="15.24" y2="21.59" width="0.4064" layer="16"/>
-<wire x1="52.07" y1="20.32" x2="52.07" y2="22.86" width="0.4064" layer="16"/>
-<wire x1="52.07" y1="22.86" x2="39.37" y2="35.56" width="0.4064" layer="16"/>
-<wire x1="15.24" y1="16.51" x2="15.24" y2="21.59" width="0" layer="19" extent="1-1"/>
+<wire x1="15.24" y1="21.59" x2="13.97" y2="21.59" width="0.4064" layer="16"/>
+<wire x1="13.97" y1="21.59" x2="12.7" y2="20.32" width="0.4064" layer="16"/>
+<wire x1="12.7" y1="20.32" x2="12.7" y2="17.78" width="0.4064" layer="16"/>
+<wire x1="12.7" y1="17.78" x2="13.97" y2="16.51" width="0.4064" layer="16"/>
+<wire x1="13.97" y1="16.51" x2="15.24" y2="16.51" width="0" layer="19" extent="1-16"/>
+<wire x1="52.07" y1="20.32" x2="52.07" y2="35.56" width="0.4064" layer="16"/>
+<wire x1="52.07" y1="35.56" x2="50.8" y2="36.83" width="0.4064" layer="16"/>
+<wire x1="50.8" y1="36.83" x2="40.64" y2="36.83" width="0.4064" layer="16"/>
+<wire x1="40.64" y1="36.83" x2="39.37" y2="35.56" width="0.4064" layer="16"/>
 </signal>
 <signal name="GND">
@@
 <contactref element="C2" pad="2"/>
 <contactref element="ESP2" pad="4"/>
-<contactref element="2SC1815" pad="1"/>
 <contactref element="18B20" pad="1"/>
 <contactref element="USB" pad="GND1"/>
-<contactref element="OPTO_PC817" pad="3"/>
 <wire x1="19.05" y1="33.02" x2="29.21" y2="33.02" width="0.4064" layer="1"/>
 <wire x1="29.21" y1="33.02" x2="44.45" y2="33.02" width="0.4064" layer="1"/>
 <wire x1="44.45" y1="33.02" x2="45.72" y2="34.29" width="0.4064" layer="1"/>
-<wire x1="45.72" y1="34.29" x2="48.26" y2="34.29" width="0.4064" layer="1"/>
 <wire x1="19.05" y1="33.02" x2="19.05" y2="25.4" width="0.4064" layer="1"/>
 <wire x1="19.05" y1="25.4" x2="17.78" y2="24.13" width="0.4064" layer="1"/>
-<wire x1="48.26" y1="34.29" x2="60.96" y2="34.29" width="0.4064" layer="1"/>
-<wire x1="60.96" y1="34.29" x2="62.23" y2="33.02" width="0.4064" layer="1"/>
-<wire x1="62.23" y1="33.02" x2="62.23" y2="24.13" width="0.4064" layer="1"/>
-<wire x1="62.23" y1="24.13" x2="62.23" y2="16.51" width="0.4064" layer="1"/>
-<wire x1="62.23" y1="16.51" x2="60.96" y2="15.24" width="0.4064" layer="1"/>
-<wire x1="60.96" y1="15.24" x2="52.07" y2="15.24" width="0.4064" layer="1"/>
-<wire x1="45.8" y1="21.56" x2="46.96" y2="21.56" width="0.4064" layer="1"/>
-<wire x1="46.96" y1="21.56" x2="49.53" y2="24.13" width="0.4064" layer="1"/>
-<wire x1="49.53" y1="24.13" x2="62.23" y2="24.13" width="0.4064" layer="1"/>
 <wire x1="3.995" y1="34.26" x2="10.13" y2="34.26" width="0.4064" layer="1"/>
 <wire x1="10.13" y1="34.26" x2="10.16" y2="34.29" width="0.4064" layer="1"/>
@@
 <wire x1="12.7" y1="34.29" x2="13.97" y2="33.02" width="0.4064" layer="1"/>
 <wire x1="13.97" y1="33.02" x2="19.05" y2="33.02" width="0.4064" layer="1"/>
-</signal>
-<signal name="N$1">
-<contactref element="R1" pad="P$1"/>
-<contactref element="2SC1815" pad="3"/>
-<contactref element="OPTO_PC817" pad="4"/>
-<wire x1="48.26" y1="29.21" x2="44.45" y2="29.21" width="0.4064" layer="1"/>
-<wire x1="44.45" y1="29.21" x2="43.18" y2="27.94" width="0.4064" layer="1"/>
-<wire x1="43.18" y1="27.94" x2="43.18" y2="25.4" width="0.4064" layer="1"/>
-<wire x1="43.18" y1="25.4" x2="44.45" y2="24.13" width="0.4064" layer="1"/>
-<wire x1="44.45" y1="24.13" x2="45.77" y2="24.13" width="0.4064" layer="1"/>
-<wire x1="45.77" y1="24.13" x2="45.8" y2="24.16" width="0.4064" layer="1"/>
+<contactref element="2SC1815" pad="1"/>
+<wire x1="45.72" y1="34.29" x2="48.26" y2="34.29" width="0.4064" layer="1"/>
+<wire x1="52.07" y1="15.24" x2="21.59" y2="15.24" width="0.4064" layer="1"/>
+<wire x1="21.59" y1="15.24" x2="20.32" y2="13.97" width="0.4064" layer="1"/>
+<wire x1="20.32" y1="13.97" x2="10.16" y2="13.97" width="0.4064" layer="1"/>
+<wire x1="10.16" y1="13.97" x2="8.89" y2="15.24" width="0.4064" layer="1"/>
+<wire x1="8.89" y1="15.24" x2="8.89" y2="33.02" width="0.4064" layer="1"/>
+<wire x1="8.89" y1="33.02" x2="10.16" y2="34.29" width="0.4064" layer="1"/>
 </signal>
 <signal name="N$2">
@@
 <wire x1="73.66" y1="34.29" x2="81.28" y2="34.29" width="0.4064" layer="1"/>
 </signal>
+<signal name="N$1">
+<contactref element="OPTO_PC817" pad="3"/>
+<contactref element="R1" pad="P$2"/>
+<wire x1="43.18" y1="35.56" x2="41.91" y2="34.29" width="0.4064" layer="16"/>
+<wire x1="41.91" y1="34.29" x2="41.91" y2="22.86" width="0.4064" layer="16"/>
+<wire x1="41.91" y1="22.86" x2="43.18" y2="21.59" width="0.4064" layer="16"/>
+<wire x1="43.18" y1="21.59" x2="45.77" y2="21.59" width="0.4064" layer="16"/>
+<wire x1="45.77" y1="21.59" x2="45.8" y2="21.56" width="0.4064" layer="16"/>
+</signal>
+<signal name="N$9">
+<contactref element="R1" pad="P$1"/>
+<contactref element="2SC1815" pad="3"/>
+<wire x1="43.18" y1="27.94" x2="46.99" y2="27.94" width="0.4064" layer="1"/>
+<wire x1="46.99" y1="27.94" x2="48.26" y2="29.21" width="0.4064" layer="1"/>
+</signal>
 </signals>
